Commit message: finish training setup

File: gym_line_follower/follower_bot.urdf (robot description, URDF)
Before this commit: robot follower, 5 links, 4 joints
Links:
- removed link caster
- removed link left_wheel
- removed link right_wheel
- added link back_left_wheel, mass 0.01; collision cylinder length=0.013 radius=0.0145; visual cylinder length=0.013 radius=0.0145
- added link back_right_wheel, mass 0.01; collision cylinder length=0.013 radius=0.0145; visual cylinder length=0.013 radius=0.0145
- added link front_left_wheel, mass 0.01; collision cylinder length=0.013 radius=0.0145; visual cylinder length=0.013 radius=0.0145
- added link front_right_wheel, mass 0.01; collision cylinder length=0.013 radius=0.0145; visual cylinder length=0.013 radius=0.0145
- added link middle_left_wheel, mass 0.01; collision cylinder length=0.013 radius=0.0145; visual cylinder length=0.013 radius=0.0145
- added link middle_right_wheel, mass 0.01; collision cylinder length=0.013 radius=0.0145; visual cylinder length=0.013 radius=0.0145
Joints:
- removed joint chassis_to_caster
- removed joint chassis_to_left_wheel
- removed joint chassis_to_right_wheel
- added joint chassis_to_back_left_wheel: type continuous, parent chassis, child back_left_wheel, origin xyz=0.0355 0.0385 -0.003 rpy=1.5708 0 0, axis 0 0 1
- added joint chassis_to_back_right_wheel: type continuous, parent chassis, child back_right_wheel, origin xyz=0.0355 -0.0385 -0.003 rpy=-1.5708 0 0, axis 0 0 -1
- added joint chassis_to_front_left_wheel: type continuous, parent chassis, child front_left_wheel, origin xyz=-0.0355 0.0385 -0.003 rpy=1.5708 0 0, axis 0 0 1
- added joint chassis_to_front_right_wheel: type continuous, parent chassis, child front_right_wheel, origin xyz=-0.0355 -0.0385 -0.003 rpy=-1.5708 0 0, axis 0 0 -1
- added joint chassis_to_middle_left_wheel: type continuous, parent chassis, child middle_left_wheel, origin xyz=0 0.042 -0.003 rpy=1.5708 0 0, axis 0 0 1
- added joint chassis_to_middle_right_wheel: type continuous, parent chassis, child middle_right_wheel, origin xyz=0 -0.042 -0.003 rpy=-1.5708 0 0, axis 0 0 -1
